File: Arming board.kicad_pcb (KiCad board)
At the start: 2 copper layers, 45 parts, among them J2 Conn_01x01_Pin, J3 Conn_01x01_Pin, J4 Conn_01x04_Pin, Q1 SQS141ELNW-T1_GE3, Q2 SQS141ELNW-T1_GE3, U1 CD40107BE, U2 TSX3702ID, U3 TSX3702ID, U6 CD40107BE

Commit message: Add files via upload
Parts:
- moved J2 50.8 mm to (68.6, 97.5), turned to 0 degrees
- moved J3 50.4 mm to (68.5, 102.5), turned to 0 degrees
- moved DZ3 47.7 mm to (64.5, 97.5)
- moved R15 45.7 mm to (51.0, 119.0)
- moved D3 44.3 mm to (55.0, 119.5), turned to 0 degrees
- moved D1 41.8 mm to (56.0, 95.0), turned to 0 degrees
- moved R5 39.5 mm to (51.0, 94.5)
- moved Q1 39.2 mm to (57.0, 78.0)
- moved F1 35.9 mm to (62.0, 90.5), turned to 0 degrees
- moved R10 34.5 mm to (50.1, 98.5)
- moved F2 34.3 mm to (62.0, 115.5), turned to 0 degrees
- moved D2 32.8 mm to (54.0, 98.5), turned to 0 degrees
- moved R9 30.9 mm to (46.5, 98.5), turned to 180 degrees
- moved Q2 26.5 mm to (57.0, 103.0)
- moved DZ2 23.8 mm to (42.0, 96.2), turned to -90 degrees
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Routing:
- net Disarm_In_1: track 0.00 -> 15.3 mm
- net Net-(U2A--): track 0.00 -> 6.21 mm
- net Net-(R10-Pad1): track 0.00 -> 1.76 mm
