File: _autosave-Arming board.kicad_pcb (KiCad board)
At the start: 2 copper layers, 46 parts, among them J2 Conn_01x01_Pin, J3 Conn_01x01_Pin, J4 Conn_01x04_Pin, Q1 SQS141ELNW-T1_GE3, Q2 SQS141ELNW-T1_GE3, U1 CD40107BE, U2 TSX3702ID, U3 TSX3702ID, U6 CD40107BE

Commit message: Add files via upload
Parts:
- removed J4: Conn_01x04_Pin, Connector_PinHeader_1.00mm:PinHeader_1x04_P1.00mm_Horizontal
- added J1: Conn_01x04_Pin, Connector_PinHeader_1.00mm:PinHeader_1x04_P1.00mm_Horizontal, F.Cu at (36.9, 102.0)
- moved C10 3.02 mm to (61.0, 111.5)
- moved R18 2.25 mm to (56.5, 107.5)
- moved F2 1.44 mm to (63.0, 116.5)
- moved U6 1.03 mm to (48.5, 106.7)
- moved F1 1.00 mm to (63.0, 90.5), turned to 180 degrees
- moved R15 0.71 mm to (50.5, 119.5), turned to 180 degrees
- moved C4 0.69 mm to (56.5, 87.5)
- moved C5 0.69 mm to (56.5, 86.5)
- moved R8 0.62 mm to (56.5, 82.5)
- moved C8 0.53 mm to (56.5, 112.2)
- moved C9 0.53 mm to (56.5, 113.2)
- moved R16 0.53 mm to (56.5, 110.7)
- moved D3 0.50 mm to (55.0, 120.0)
- moved R7 0.48 mm to (56.5, 84.5)
Routing:
- net /Arm_In_1: track 0.00 -> 43.4 mm, vias 0 -> 2
- net GND: track 0.00 -> 39.5 mm, vias 0 -> 5
- net /Arming logic 1/-out: track 0.00 -> 25.5 mm
- net Net-(U1-A): track 0.00 -> 18.4 mm
- net VCC: track 0.00 -> 13.0 mm
- net Net-(U1-E): track 0.00 -> 10.8 mm, vias 0 -> 2
- net Net-(D3-K): track 0.00 -> 7.59 mm
- net /Disarm_In_1: track 15.3 -> 22.2 mm
- net Net-(U3A--): track 0.00 -> 6.52 mm
- net /Arming logic 1/out: track 0.00 -> 6.24 mm
Other:
- copper layers 2 -> 4
