File: Arming logic.kicad_sch (KiCad schematic)
At the start: 17 parts, among them U1 CD40107BE, U2 TSX3702ID, U3 TSX3702ID

Commit message: Add files via upload
Parts:
- removed U3: TSX3702ID, PCM_Package_SO_AKL:SO-8_3.9x4.9mm_P1.27mm, symbol PCM_Analog_Comparator_AKL:TSX3702ID
- added unit 2 of U2
- C1, C2: value C -> 1u; footprint (none) -> Capacitor_SMD:C_0402_1005Metric
- C3, C4, C5: value C -> 100n; footprint (none) -> Capacitor_SMD:C_0402_1005Metric
- D1: value D -> 4.7; footprint (none) -> Diode_SMD:D_SOD-123
- R1, R2, R3, R4, R5, R6, R7, R8: value R -> 10k; footprint (none) -> Resistor_SMD:R_0402_1005Metric
- U1: footprint CD40107BE:DIP794W45P254L959H508Q8 -> cd40107:DIP794W45P254L959H508Q8
Connections:
- net at D1.1 (K), R5.2, U2.3 (+): now also U2.5 (+)
- net at C2.1, R3.2, R4.1: now also U2.6 (-)
- net at U1.6 (E): now also U2.7
- net power_fused renamed pwr_fused

Commit message: Add files via upload
Parts:
- C1: footprint Capacitor_SMD:C_0402_1005Metric -> (none)
- R2: footprint Resistor_SMD:R_0402_1005Metric -> (none)
Connections:
- no-connect marks 0 -> 1

Commit message: Add files via upload
Parts:
- C1: footprint (none) -> Capacitor_SMD:C_0402_1005Metric
- R2: footprint (none) -> Resistor_SMD:R_0402_1005Metric
Changed lines of the file:
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@@
 			)
 		)
-		(property "Footprint" ""
+		(property "Footprint" "Resistor_SMD:R_0402_1005Metric"
 			(at 85.852 77.47 90)
 			(effects
@@
 			)
 		)
-		(property "Footprint" ""
+		(property "Footprint" "Capacitor_SMD:C_0402_1005Metric"
 			(at 98.7552 81.28 0)
 			(effects

Commit message: continued scematic
Changed lines of the file:
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@@
+	(wire
+		(pts
+			(xy 87.63 129.54) (xy 87.63 125.73)
+		)
+		(stroke
+			(width 0)
+			(type default)
+		)
+	)
 	(wire
 		(pts
@@
 	(symbol
 		(lib_id "power:GND")
-		(at 87.63 125.73 0)
+		(at 87.63 129.54 0)
 		(unit 1)
 		(exclude_from_sim no)
@@
 		(fields_autoplaced yes)
 		(property "Reference" "#PWR02"
-			(at 87.63 132.08 0)
+			(at 87.63 135.89 0)
 			(effects
 				(font
@@
 		)
 		(property "Value" "GND"
-			(at 87.63 130.81 0)
+			(at 87.63 134.62 0)
 			(effects
 				(font
@@
 		)
 		(property "Footprint" ""
-			(at 87.63 125.73 0)
+			(at 87.63 129.54 0)
 			(effects
 				(font
@@
 		)
 		(property "Datasheet" ""
-			(at 87.63 125.73 0)
+			(at 87.63 129.54 0)
 			(effects
 				(font
@@
 		)
 		(property "Description" "Power symbol creates a global label with name \"GND\" , ground"
-			(at 87.63 125.73 0)
-			(effects
-				(font
+			(at 87.63 129.54 0)
+			(effects
+				(font
